File: PCB_Schematic_ECE477.brd (EAGLE design)
At the start: 100 x 80 mm, 21 parts, among them U1 STM32F107VCT6, U2 OKI-78SR_3V3_SMPS

Commit message: Updated PCB
Parts:
- removed C1, C2: (no value), resistor:C025-024X044
- removed G1: AB9V, battery:AB9V
- removed PAD1, PAD2, PAD3, PAD4: (no value), wirepad:1,6/0,8
- removed SV1, SV4, SV5, SV8: (no value), con-lstb:MA04-2
- removed SV2, SV3: (no value), con-lstb:MA06-2
- removed SV7: (no value), con-lstb:MA08-2
- added C3, C4: 1uF, SparkFun-Passives:1206
- added C5: (no value), SparkFun-Passives:1206
- added JP1, JP2, JP3: (no value), SparkFun-Connectors:1X04
- added JP4, JP5, JP8: (no value), SparkFun-Connectors:1X06
- added JP6: (no value), SparkFun-Connectors:1X08
- added JP7: (no value), SparkFun-Connectors:1X10
- added R10, R11, R12, R13, R4, R5, R6, R7, R8, R9: 10k, SparkFun-Resistors:1206
- added R14: (no value), SparkFun-Resistors:1206
- added R16: 10K, SparkFun-Resistors:1206
- added S1: 5501, switch:5501
- added U$2: MUX_DEVMUX_VAR_1, QSOP28:QSOP28
- added U$3, U$4, U$5, U$6, U$7, U$8: BSS138, BSS138:BSS138
- added X1: 87758-0216, con-molex:87758-0216
- R1: value (none) -> 10K; device rcl:0204V -> SparkFun-Resistors:1206
- R2, R3: value (none) -> 10k; device rcl:0204V -> SparkFun-Resistors:1206
- moved R2 61.3 mm to (67.3, 48.3)
- moved R3 55.8 mm to (59.7, 48.3)
- moved U2 38.1 mm to (8.89, 14.0)
- moved R1 16.5 mm to (3.81, 54.6)
- moved U$1 16.5 mm to (29.2, 14.0)
- moved XB1 7.18 mm to (86.4, 20.3)
- moved U1 2.84 mm to (50.8, 24.1), turned to 90 degrees
Connections:
- net VDDA renamed PA0-WKUP
- net VDD_4 renamed PA4
- net VREF- renamed VREF+
- removed net N$1: G1.+, U1.27, U2.VIN
- removed net N$10: SV2.8, U1.8
- removed net N$12: SV2.4, U1.47
- removed net N$13: SV3.12, U1.97
- removed net N$14 (its old number): SV3.10, U1.98
- removed net N$15: SV3.8, U1.9
- removed net N$25: R1.2, U$1.2
- new net HV: C3.1, JP1.3, JP2.1, JP3.2, JP4.1, JP5.6, JP6.8, JP7.10, R1.2, R11.2, R12.2, R13.2, R16.2, R3.2, R5.2, R9.2, U$1.3, U2.VOUT
- new net HV1: R10.1, U$4.S, U1.70
- new net HV2: JP3.3, R3.1, U$3.D
- new net HV3: JP4.3, R12.1, U$6.D
- new net HV4: JP4.4, R13.1, U$7.D
- new net HV5: JP5.1, R9.1, U$5.D
- new net HV6: JP3.4, R5.1, U$8.D
- new net LV: R10.2, R2.2, R4.2, R6.2, R7.2, R8.2, U$3.G, U$4.G, U$5.G, U$6.G, U$7.G, U$8.G
- new net LV1: JP2.3, R11.1, U$4.D
- new net LV2: R2.1, U$3.S, U1.59
- new net LV3: R6.1, U$6.S, U1.46
- new net LV4: R7.1, U$7.S, U1.47
- new net LV5: R8.1, U$5.S, U1.55
- new net LV6: R4.1, U$8.S, U1.60
- new net N$10_NTJRST: JP7.7, U1.90
- new net N$10_TCLK: JP7.6, U1.76
- new net N$10_TDI: JP7.3, U1.77
- new net N$10_TDO: JP7.5, U1.89
- new net N$10_TMS: JP7.4, U1.72
- new net N$24: U$2.7, U1.43
- new net N$26: U$2.10, U1.44
- new net N$27: U$2.18, U1.63
- new net N$28: U$2.21, U1.64
- new net N$29: JP8.1, U$2.2
- new net N$3: JP6.6, U$2.19
- new net N$30: JP8.2, U$2.5
- new net N$31: JP8.3, U$2.8
- new net N$32: JP8.4, U$2.11
- new net N$33: JP8.5, U$2.17
- new net N$34: JP8.6, U$2.20
- new net N$35: JP6.1, U$2.3
- new net N$41: JP6.4, U$2.12
- new net N$42: JP6.5, U$2.16
- new net RESET_OUT: C5.2, JP5.3, JP7.2, R14.2, S1.1B, U1.14, XB1.5
- new net VIN_MICRO_3.3: C4.1, JP7.1, R14.1, U$1.2, U$1.4, U1.100, U1.11, U1.21, U1.27, U1.50, U1.75, XB1.1
- net GND: now also C3.2, C4.2, C5.1, JP1.4, JP2.4, JP3.1, JP4.6, JP5.5, JP6.7, S1.NO, U$2.14, U$2.28, X1.2; no longer C1.2, C2.2, G1.-, R1.1, SV1.2, SV2.2, SV3.4, SV4.2, SV5.8, SV7.4, SV8.2
- net N$11: now also U2.VIN, X1.1; no longer SV2.6, U1.46
- net N$2: now also JP2.2, U1.69; no longer C1.1, R2.2, R3.2, SV1.8, SV2.12, SV3.2, SV4.4, SV5.6, SV7.2, SV8.4, U$1.3, U2.VOUT
- net N$20: now also U$2.13; no longer SV4.8
- net N$21: now also U$2.15, U1.17; no longer SV4.6, U1.15
- net N$22: now also U$2.1, U1.39; no longer SV5.4, U1.78
- net N$23: now also U$2.4, U1.41; no longer SV5.2, U1.79
- net N$4: now also JP1.2; no longer SV8.6
- net N$5: now also JP6.2, U$2.6; no longer C2.1, U$1.4, U1.100, U1.11, U1.21, U1.50, U1.75, XB1.1
- net N$6: now also JP6.3, U$2.9; no longer SV1.6, U1.38
- net N$7: now also JP1.1, R1.1, R16.1; no longer R2.1, R3.1, SV8.8
- net N$8: now also JP5.2, U1.56; no longer SV1.4, U1.37
- net N$9: now also JP4.2; no longer SV2.10
Routing:
- net HV: track 0.00 -> 287.0 mm, vias 0 -> 5
- net N$2: track 242.0 -> 51.7 mm
- net RESET_OUT: track 0.00 -> 176.0 mm
- net N$1: track 132.8 -> 0.00 mm, vias 0 -> 1
- net VIN_MICRO_3.3: track 0.00 -> 123.2 mm, vias 0 -> 7
- net N$5: track 163.8 -> 46.6 mm, vias 0 -> 2
- net LV: track 0.00 -> 116.9 mm, vias 0 -> 2
- net N$12: track 90.2 -> 0.00 mm
- net N$11: track 96.1 -> 12.7 mm
- net N$10_TMS: track 0.00 -> 82.2 mm, vias 0 -> 2
- net N$15: track 71.0 -> 0.00 mm
- net N$6: track 105.3 -> 37.6 mm, vias 0 -> 1
- net LV3: track 0.00 -> 63.4 mm, vias 0 -> 9
- net N$8: track 99.7 -> 37.7 mm, vias 0 -> 1
- net HV6: track 0.00 -> 59.9 mm, vias 0 -> 3
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Other:
- board size 100 x 80 mm -> 100 x 61 mm

Commit message: Latest Schematics
Parts:
- removed S1: 5501, switch:5501
- added C1, C2, C6, C7, C8, C9: (no value), SparkFun-Passives:1206
- added H1, H2, H3, H4: MOUNT-HOLE2.8, holes:2,8
- added LED2: (no value), eagle-ltspice:LED_1206
- added U$9: CUSTOM_SWITCH_DEVICE, custom_switch:CUSTOM_SWITCH_PACKAGE
- moved JP6 86.1 mm to (27.9, 3.81), turned to 0 degrees
- moved JP2 79.8 mm to (95.2, 43.2), turned to 90 degrees
- moved R11 79.0 mm to (90.2, 44.5), turned to 90 degrees
- moved R10 73.7 mm to (90.2, 49.5), turned to 90 degrees
- moved U$4 73.7 mm to (86.4, 44.5)
- moved JP8 56.9 mm to (52.1, 3.81)
- moved JP7 54.8 mm to (33.0, 58.4)
- moved U$2 47.3 mm to (40.6, 20.3), turned to 0 degrees
- moved U$3 42.0 mm to (20.3, 47.6)
- moved R3 32.4 mm to (91.4, 54.6)
- moved U$5 22.8 mm to (66.7, 54.6)
- moved R8 22.5 mm to (73.0, 54.0)
- moved JP3 21.7 mm to (81.3, 58.4)
- moved JP5 21.7 mm to (62.2, 58.4)
- moved R5 19.8 mm to (79.4, 54.6)
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Connections:
- net PA0-WKUP renamed N$55
- net PA4 renamed N$87
- net VREF+ renamed N$53
- removed net VBAT: U1.6
- new net N$1: C8.2, U1.73
- new net N$10: C9.2, U1.48
- new net N$12: U1.23
- new net N$13: U1.24
- new net N$15: U1.25
- new net N$19: U1.29
- new net N$25: U1.30
- new net N$36: U1.31
- new net N$37: U1.32
- new net N$38: U1.67
- new net N$39: U1.68
- new net N$43: U1.35
- new net N$44: U1.36
- new net N$45: U1.37
- new net N$46: U1.91
- new net N$47: U1.92
- new net N$48: U1.93
- new net N$49: U1.51
- new net N$50: U1.52
- new net N$51: U1.53
- new net N$52: U1.54
- new net N$54: U1.94
- new net N$56: U1.12
- new net N$57: U1.13
- new net N$58: U1.45
- new net N$59: U1.42
- new net N$60: U1.38
- new net N$61: U1.5
- new net N$62: U1.4
- new net N$63: U1.3
- new net N$64: U1.2
- new net N$65: U1.1
- new net N$66: U1.98
- new net N$67: U1.97
- new net N$68: U1.62
- new net N$69: U1.61
- new net N$70: U1.58
- new net N$71: U1.57
- new net N$72: U1.88
- new net N$73: U1.87
- new net N$74: U1.86
- new net N$75: U1.85
- new net N$76: U1.84
- new net N$77: U1.82
- new net N$78: U1.81
- new net N$79: U1.9
- new net N$80: U1.8
- new net N$81: U1.79
- new net N$82: U1.78
- new net N$83: U1.34
- new net N$84: U1.33
- new net N$85: U1.18
- new net N$86: U1.15
- net GND: now also C1.2, C2.2, C6.2, C7.2, C8.1, C9.1, LED2.C, U$9.P$2; no longer S1.NO
- net RESET_OUT: now also U$9.P$1; no longer S1.1B
- net VIN_MICRO_3.3: now also C1.1, C2.1, C6.1, C7.1, LED2.A, U1.6
Routing:
- net LV2: track 10.9 -> 106.1 mm, vias 2 -> 4
- net VIN_MICRO_3.3: track 123.2 -> 195.6 mm, vias 7 -> 11
- net HV2: track 18.0 -> 89.9 mm, vias 0 -> 1
- net N$27: track 0.00 -> 47.9 mm, vias 0 -> 2
- net N$3: track 13.7 -> 58.4 mm
- net N$10_TMS: track 82.2 -> 39.6 mm
- net N$26: track 0.00 -> 39.0 mm, vias 0 -> 4
- net N$21: track 69.5 -> 35.2 mm, vias 5 -> 2
- net HV6: track 59.9 -> 25.9 mm, vias 3 -> 1
- net N$9: track 96.9 -> 67.0 mm, vias 10 -> 3
- net RESET_OUT: track 176.0 -> 146.2 mm, vias 0 -> 7
- net LV6: track 13.8 -> 43.4 mm, vias 1 -> 4
- net N$42: track 14.5 -> 42.9 mm, vias 0 -> 4
- net N$18: track 76.5 -> 50.6 mm, vias 4 -> 3
- net N$34: track 16.4 -> 41.8 mm, vias 1 -> 2
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Other:
- board size 100 x 61 mm -> 100 x 63.5 mm
