File: PCB_Schematic_ECE477.sch (EAGLE design)
At the start: 21 parts, among them U1 STM32F107VCT6, U2 OKI-78SR_3V3_SMPS

Commit message: Updated PCB
Parts:
- removed C1, C2: (no value), resistor:C-US025-024X044
- removed G1: AB9V, battery:AB9V
- removed PAD1, PAD2, PAD3, PAD4: (no value), wirepad:1,6/0,8
- removed SV1, SV4, SV5, SV8: (no value), con-lstb:MA04-2
- removed SV2, SV3: (no value), con-lstb:MA06-2
- removed SV7: (no value), con-lstb:MA08-2
- added C3, C4: 1uF, SparkFun-Passives:CAP1206
- added C5: (no value), SparkFun-Passives:CAP1206
- added JP1, JP2, JP3: (no value), SparkFun-Connectors:M04PTH
- added JP4, JP5, JP8: (no value), SparkFun-Connectors:M06SILK_FEMALE_PTH
- added JP6: (no value), SparkFun-Connectors:M08SILK_FEMALE_PTH
- added JP7: (no value), SparkFun-Connectors:M10SILK_FEMALE_PTH
- added R10, R11, R12, R13, R4, R5, R6, R7, R8, R9: 10k, SparkFun-Resistors:RESISTOR1206
- added R14: (no value), SparkFun-Resistors:RESISTOR1206
- added R16: 10K, SparkFun-Resistors:RESISTOR1206
- added S1: 5501, switch:5501
- added U$2: MUX_DEVMUX_VAR_1, QSOP28:MUX_DEVMUX_VAR_1
- added U$3, U$4, U$5, U$6, U$7, U$8: BSS138, BSS138:BSS138
- added X1: 87758-0216, con-molex:87758-0216
- R1: value (none) -> 10K; device rcl:R-US_0204/2V -> SparkFun-Resistors:RESISTOR1206
- R2, R3: value (none) -> 10k; device rcl:R-US_0204/2V -> SparkFun-Resistors:RESISTOR1206
Connections:
- removed net N$1: G1.+, U1.VSS_4, U2.VIN
- removed net N$10: SV2.8, U1.PC14-OSC32_IN
- removed net N$12: SV2.4, U1.PB10
- removed net N$13: SV3.12, U1.PE0
- removed net N$14 (its old number): SV3.10, U1.PE1
- removed net N$15: SV3.8, U1.PC15-OSC32_OUT
- removed net N$25: R1.2, U$1.OUTPUT_2
- new net HV: C3.1, JP1.3, JP2.1, JP3.2, JP4.1, JP5.6, JP6.8, JP7.10, R1.2, R11.2, R12.2, R13.2, R16.2, R3.2, R5.2, R9.2, U$1.INPUT, U2.VOUT
- new net HV1: R10.1, U$4.S, U1.PA_11
- new net HV2: JP3.3, R3.1, U$3.D
- new net HV3: JP4.3, R12.1, U$6.D
- new net HV4: JP4.4, R13.1, U$7.D
- new net HV5: JP5.1, R9.1, U$5.D
- new net HV6: JP3.4, R5.1, U$8.D
- new net LV: R10.2, R2.2, R4.2, R6.2, R7.2, R8.2, U$3.G, U$4.G, U$5.G, U$6.G, U$7.G, U$8.G
- new net LV1: JP2.3, R11.1, U$4.D
- new net LV2: R2.1, U$3.S, U1.PD12
- new net LV3: R6.1, U$6.S, U1.PB10
- new net LV4: R7.1, U$7.S, U1.PB11
- new net LV5: R8.1, U$5.S, U1.PD8
- new net LV6: R4.1, U$8.S, U1.PD13
- new net N$10_NTJRST: JP7.7, U1.PB4
- new net N$10_TCLK: JP7.6, U1.PA14
- new net N$10_TDI: JP7.3, U1.PA15
- new net N$10_TDO: JP7.5, U1.PB3
- new net N$10_TMS: JP7.4, U1.PA_13
- new net N$24: U$2.P$7, U1.PE13
- new net N$26: U$2.P$10, U1.PE14
- new net N$27: U$2.P$18, U1.PC6
- new net N$28: U$2.P$21, U1.PC7
- new net N$29: JP8.1, U$2.P$2
- new net N$3: JP6.6, U$2.P$19
- new net N$30: JP8.2, U$2.P$5
- new net N$31: JP8.3, U$2.P$8
- new net N$32: JP8.4, U$2.P$11
- new net N$33: JP8.5, U$2.P$17
- new net N$34: JP8.6, U$2.P$20
- new net N$35: JP6.1, U$2.P$3
- new net N$41: JP6.4, U$2.P$12
- new net N$42: JP6.5, U$2.P$16
- new net RESET_OUT: C5.2, JP5.3, JP7.2, R14.2, S1.1B, U1.NRST, XB1.!RESET
- new net VIN_MICRO_3.3: C4.1, JP7.1, R14.1, U$1.OUTPUT, U1.VDD4, U1.VDDA, U1.VDD_1, U1.VDD_2, U1.VDD_3, U1.VDD_5, XB1.VCC
- net GND: now also C3.2, C4.2, C5.1, JP1.4, JP2.4, JP3.1, JP4.6, JP5.5, JP6.7, S1.NO, U$2.P$14, U$2.P$28, U1.VSS4, X1-2.S; no longer C1.2, C2.2, G1.-, R1.1, SV1.2, SV2.2, SV3.4, SV4.2, SV5.8, SV7.4, SV8.2, U1.PA3
- net N$11: now also U2.VIN, X1-1.S; no longer SV2.6, U1.PE15
- net N$2: now also JP2.2, U1.PA_10; no longer C1.1, R2.2, R3.2, SV1.8, SV2.12, SV3.2, SV4.4, SV5.6, SV7.2, SV8.4, U$1.INPUT, U2.VOUT
- net N$20: now also U$2.P$13; no longer SV4.8
- net N$21: now also U$2.P$15, U1.PC2; no longer SV4.6, U1.PC0
- net N$22: now also U$2.P$1, U1.PE9; no longer SV5.4, U1.PC10
- net N$23: now also U$2.P$4, U1.PE11; no longer SV5.2, U1.PC11
- net N$4: now also JP1.2; no longer SV8.6
- net N$5: now also JP6.2, U$2.P$6; no longer C2.1, U$1.OUTPUT, U1.VDD_1, U1.VDD_2, U1.VDD_3, U1.VDD_5, U1.VREF+, XB1.VCC
- net N$6: now also JP6.3, U$2.P$9; no longer SV1.6, U1.PE7
- net N$7: now also JP1.1, R1.1, R16.1; no longer R2.1, R3.1, SV8.8
- net N$8: now also JP5.2, U1.PD9; no longer SV1.4, U1.PB2
- net N$9: now also JP4.2; no longer SV2.10
Other:
- moved on the sheet: R1, R2, R3

Commit message: Latest Schematics
Parts:
- removed S1: 5501, switch:5501
- added C1, C2, C6, C7, C8, C9: (no value), SparkFun-Passives:CAP1206
- added H1, H2, H3, H4: MOUNT-HOLE2.8, holes:MOUNT-HOLE2.8
- added LED2: (no value), eagle-ltspice:LED_E
- added U$9: CUSTOM_SWITCH_DEVICE, custom_switch:CUSTOM_SWITCH_DEVICE
Connections:
- new net N$1: C8.2, U1.VCAP2
- new net N$10: C9.2, U1.VCAP1
- new net N$12: U1.PA1
- new net N$13: U1.PA2
- new net N$15: U1.PA3
- new net N$19: U1.PA5
- new net N$25: U1.PA6
- new net N$36: U1.PA7
- new net N$37: U1.PC4
- new net N$38: U1.PA_8
- new net N$39: U1.PA_9
- new net N$43: U1.PB1
- new net N$44: U1.PB2
- new net N$45: U1.PE7
- new net N$46: U1.PB5
- new net N$47: U1.PB6
- new net N$48: U1.PB7
- new net N$49: U1.PB12
- new net N$50: U1.PB13
- new net N$51: U1.PB14
- new net N$52: U1.PB15
- new net N$53: U1.VREF+
- new net N$54: U1.BOOT0
- new net N$55: U1.PA0-WKUP
- new net N$56: U1.OSC_IN
- new net N$57: U1.OSC_OUT
- new net N$58: U1.PE15
- new net N$59: U1.PE12
- new net N$60: U1.PE8
- new net N$61: U1.PE6
- new net N$62: U1.PE5
- new net N$63: U1.PE4
- new net N$64: U1.PE3
- new net N$65: U1.PE2
- new net N$66: U1.PE1
- new net N$67: U1.PE0
- new net N$68: U1.PD15
- new net N$69: U1.PD14
- new net N$70: U1.PD11
- new net N$71: U1.PD10
- new net N$72: U1.PD7
- new net N$73: U1.PD6
- new net N$74: U1.PD5
- new net N$75: U1.PD4
- new net N$76: U1.PD3
- new net N$77: U1.PD1
- new net N$78: U1.PD0
- new net N$79: U1.PC15-OSC32_OUT
- new net N$80: U1.PC14-OSC32_IN
- new net N$81: U1.PC11
- new net N$82: U1.PC10
- new net N$83: U1.PB0
- new net N$84: U1.PC5
- new net N$85: U1.PC3
- new net N$86: U1.PC0
- new net N$87: U1.PA4
- net GND: now also C1.2, C2.2, C6.2, C7.2, C8.1, C9.1, LED2.C, U$2.GND, U$2.VCC, U$9.P$2; no longer S1.NO, U$2.P$14, U$2.P$28
- net N$20: now also U$2.AEN; no longer U$2.P$13
- net N$21: now also U$2.BEN; no longer U$2.P$15
- net N$22: now also U$2.A0; no longer U$2.P$1
- net N$23: now also U$2.A1; no longer U$2.P$4
- net N$24: now also U$2.A2; no longer U$2.P$7
- net N$26: now also U$2.A3; no longer U$2.P$10
- net N$27: now also U$2.A4; no longer U$2.P$18
- net N$28: now also U$2.A5; no longer U$2.P$21
- net N$29: now also U$2.B0; no longer U$2.P$2
- net N$3: now also U$2.AB5; no longer U$2.P$19
- net N$30: now also U$2.B1; no longer U$2.P$5
- net N$31: now also U$2.B2; no longer U$2.P$8
- net N$32: now also U$2.B3; no longer U$2.P$11
- net N$33: now also U$2.B4; no longer U$2.P$17
- net N$34: now also U$2.B5; no longer U$2.P$20
- net N$35: now also U$2.AB0; no longer U$2.P$3
- net N$41: now also U$2.AB3; no longer U$2.P$12
- net N$42: now also U$2.AB4; no longer U$2.P$16
- net N$5: now also U$2.AB1; no longer U$2.P$6
- net N$6: now also U$2.AB2; no longer U$2.P$9
- net RESET_OUT: now also U$9.P$1; no longer S1.1B
- net VIN_MICRO_3.3: now also C1.1, C2.1, C6.1, C7.1, LED2.A, U1.VBAT
